Commit message: practica09

File: catkin_ws/src/hardware/justina_description/urdf/justina_base.xacro (robot description, xacro)
@@ -206,5 +206,5 @@
   </link>
   <joint name="laser_connect" type="fixed">
-    <origin xyz="0.17 0 0.44" />
+    <origin xyz="0.17 0 1.44" rpy="1.5708 0 0" />
     <parent link="base_link"/>
     <child link="laser_link"/>

Commit message: correcion Practica9

File: catkin_ws/src/hardware/justina_description/urdf/justina_base.xacro (robot description, xacro)
@@ -206,5 +206,5 @@
   </link>
   <joint name="laser_connect" type="fixed">
-    <origin xyz="0.17 0 1.44" rpy="1.5708 0 0" />
+    <origin xyz="0.17 0 0.44" />
     <parent link="base_link"/>
     <child link="laser_link"/>
