Commit message: Update packages and readme

File: catkin_ws/src/hardware/justina_description/urdf/justina_right_arm.xacro (robot description, xacro)
@@ -9,5 +9,5 @@
         <box size = "0.04025 0.108 0.065"/>
       </geometry>
-      <material name = "ra_material"><color rgba="1.0 0.5 0 1"/></material>
+      <material name = "ra_material_red"><color rgba="1.0 0 0 1"/></material>
     </visual>
     <collision>
@@ -32,5 +32,5 @@
         <box size = "0.04025 0.06 0.04025"/>
       </geometry>
-      <material name = "ra_material"><color rgba="1.0 0.5 0 1"/></material>
+      <material name = "ra_material_orange"><color rgba="1.0 0.5 0 1"/></material>
     </visual>
     <collision>
@@ -55,5 +55,5 @@
         <box size = "0.04025 0.04025 0.19"/>
       </geometry>
-      <material name = "ra_material"><color rgba="1.0 0.5 0 1"/></material>
+      <material name = "ra_material_yellow"><color rgba="1.0 1 0 1"/></material>
     </visual>
     <visual>
@@ -62,5 +62,5 @@
         <box size = "0.06 0.04025 0.04025"/>
       </geometry>
-      <material name = "la_material"><color rgba="1.0 0.5 0 1"/></material>
+      <material name = "la_material_yellow"><color rgba="1.0 1 0 1"/></material>
     </visual>
     <collision>
@@ -89,12 +89,12 @@
       <origin xyz="0 0 -0.04" rpy = "0 0 0"/>
       <geometry>
-        <box size = "0.04025 0.04025 0.06"/>
-      </geometry>
-      <material name = "ra_material"><color rgba="1.0 0.5 0 1"/></material>
+        <box size = "0.04025 0.04025 0.05"/>
+      </geometry>
+      <material name = "ra_material_green"><color rgba="0 0.5 0 1"/></material>
     </visual>
     <collision>
       <origin xyz="0 0 -0.04" rpy = "0 0 0"/>
       <geometry>
-        <box size = "0.04025 0.04025 0.06"/>
+        <box size = "0.04025 0.04025 0.05"/>
       </geometry>
     </collision>
@@ -110,29 +110,29 @@
   <link name="right_arm_link4">
     <visual>
-      <origin xyz="0 0 -0.11" rpy = "0 0 0"/>
-      <geometry>
-        <box size = "0.04025 0.04025 0.16"/>
-      </geometry>
-      <material name = "ra_material"><color rgba="1.0 0.5 0 1"/></material>
-    </visual>
-    <visual>
+      <origin xyz="0 0 -0.075" rpy = "0 0 0"/>
+      <geometry>
+        <box size = "0.04025 0.04025 0.08"/>
+      </geometry>
+      <material name = "ra_material_blue"><color rgba="0 0 1 1"/></material>
+    </visual>
+    <!--<visual>
       <origin xyz="-0.01 0 -0.167" rpy = "0 0 0"/>
       <geometry>
+        <box size = "0.06 -0.04025 0.04025"/>
+      </geometry>
+      <material name = "la_material_blue"><color rgba="0 0 1 1"/></material>
+    </visual> -->
+    <collision>
+      <origin xyz="0 0 -0.075" rpy = "0 0 0"/>
+      <geometry>
+        <box size = "0.04025 0.04025 0.08"/>
+      </geometry>
+    </collision>
+    <!--<collision>
+      <origin xyz="-0.01 0 -0.167" rpy = "0 0 0"/>
+      <geometry>
         <box size = "0.06 0.04025 0.04025"/>
       </geometry>
-      <material name = "la_material"><color rgba="1.0 0.5 0 1"/></material>
-    </visual>
-    <collision>
-      <origin xyz="0 0 -0.11" rpy = "0 0 0"/>
-      <geometry>
-        <box size = "0.04025 0.04025 0.16"/>
-      </geometry>
-    </collision>
-    <collision>
-      <origin xyz="-0.01 0 -0.167" rpy = "0 0 0"/>
-      <geometry>
-        <box size = "0.06 0.04025 0.04025"/>
-      </geometry>
-    </collision>
+    </collision> -->
     <inertial>
       <origin xyz="-0.01 0 -0.147" rpy = "0 0 0"/>
@@ -146,18 +146,18 @@
   <link name="right_arm_link5">
     <visual>
+      <origin xyz="0.02 0 0.005" rpy = "0 0 0"/>
+      <geometry>
+        <box size = "0.07 0.03025 0.05"/>
+      </geometry>
+      <material name = "ra_material_purple"><color rgba="1.0 0 1 1"/></material>
+    </visual>
+    <collision>
+      <origin xyz="0.02 0 0.005" rpy = "0 0 0"/>
+      <geometry>
+        <box size = "0.07 0.03025 0.05"/>
+      </geometry>
+    </collision>
+    <inertial>
       <origin xyz="0 0 -0.025" rpy = "0 0 0"/>
-      <geometry>
-        <box size = "0.04025 0.04025 0.02"/>
-      </geometry>
-      <material name = "ra_material"><color rgba="1.0 0.5 0 1"/></material>
-    </visual>
-    <collision>
-      <origin xyz="0 0 -0.025" rpy = "0 0 0"/>
-      <geometry>
-        <box size = "0.04025 0.04025 0.02"/>
-      </geometry>
-    </collision>
-    <inertial>
-      <origin xyz="0 0 -0.025" rpy = "0 0 0"/>
       <mass value="0.125"/>
       <inertia
@@ -169,18 +169,31 @@
   <link name="right_arm_link6">
     <visual>
+      <origin xyz="0.02 0 -0.045" rpy = "0 0 0"/>
+      <geometry>
+        <box size = "0.07025 0.04025 0.02"/>
+      </geometry>
+      <material name = "ra_material_red"><color rgba="1.0 0 0 1"/></material>
+    </visual>
+    <visual>
+      <origin xyz="0 0 -0.088" rpy="0 0 0"/>
+      <geometry>
+        <box size = "0.03025 0.04025 0.03"/>
+      </geometry>
+      <material name ="ra_material_red"><color rgba= "1.0 0 0 1 "/></material>
+    </visual>
+    <collision>
+      <origin xyz="0.02 0 -0.045" rpy = "0 0 0"/>
+      <geometry>
+        <box size = "0.07025 0.04025 0.02"/>
+      </geometry>
+    </collision>
+    <collision>
+      <origin xyz="0 0 -0.088" rpy="0 0 0"/>
+      <geometry>
+        <box size = "0.03025 0.04025 0.03"/>
+      </geometry>
+    </collision>
+    <inertial>
       <origin xyz="0 0 -0.042" rpy = "0 0 0"/>
-      <geometry>
-        <box size = "0.04025 0.04025 0.04"/>
-      </geometry>
-      <material name = "ra_material"><color rgba="1.0 0.5 0 1"/></material>
-    </visual>
-    <collision>
-      <origin xyz="0 0 -0.042" rpy = "0 0 0"/>
-      <geometry>
-        <box size = "0.04025 0.04025 0.04"/>
-      </geometry>
-    </collision>
-    <inertial>
-      <origin xyz="0 0 -0.042" rpy = "0 0 0"/>
       <mass value="0.125"/>
       <inertia
@@ -191,24 +204,24 @@
   </link>
   <link name="right_arm_link7">
-    <visual>
+   <!-- <visual>
+      <origin xyz="-0.025 0 -0.03" rpy = "0 0 0"/>
+      <geometry>
+        <box size = "0.11 0.03525 0.03525"/>
+      </geometry>
+      <material name = "ra_material_or"><color rgba="1 0.5 0 1"/></material>
+    </visual>-->
+    <visual>
+      <origin xyz="0 0 -0.055" rpy = "0 0 0"/>
+      <geometry>
+        <box size = "0.03 0.1 0.03"/>
+      </geometry>
+      <material name = "ra_material_green"><color rgba="0 0.5 0 1"/></material>
+    </visual>
+    <!--<collision>
       <origin xyz="-0.01 0 -0.03" rpy = "0 0 0"/>
       <geometry>
         <box size = "0.06 0.03525 0.03525"/>
       </geometry>
-      <material name = "ra_material"><color rgba="1.0 0.5 0 1"/></material>
-    </visual>
-    <visual>
-      <origin xyz="0 0 -0.055" rpy = "0 0 0"/>
-      <geometry>
-        <box size = "0.03 0.1 0.03"/>
-      </geometry>
-      <material name = "ra_material"><color rgba="1.0 0.5 0 1"/></material>
-    </visual>
-    <collision>
-      <origin xyz="-0.01 0 -0.03" rpy = "0 0 0"/>
-      <geometry>
-        <box size = "0.06 0.03525 0.03525"/>
-      </geometry>
-    </collision>
+    </collision>-->
     <collision>
       <origin xyz="0 0 -0.055" rpy = "0 0 0"/>
@@ -298,5 +311,5 @@
   </joint>
   <joint name="ra_4_joint" type="revolute">
-    <origin xyz="0.005 0.0 -0.013" rpy="0 0 0"/>
+    <origin xyz="0 0.0 -0.035" rpy="0 0 0"/>
     <parent link="right_arm_link3"/>
     <child link="right_arm_link4"/>
@@ -306,21 +319,21 @@
   </joint>
   <joint name="ra_5_joint" type="revolute">
-    <origin xyz="0 0.0 -0.18" rpy="0 0 0"/>
+    <origin xyz="0 0.0 -0.15" rpy="0 0 0"/>
     <parent link="right_arm_link4"/>
     <child link="right_arm_link5"/>
-    <axis xyz="0 0 1" />
+    <axis xyz="0 -1 0" />
     <dynamics damping ="0.1" />
     <limit effort="6.0" velocity="3.0" lower="-2.5" upper="2.5"/>
   </joint>
   <joint name="ra_6_joint" type="revolute">
-    <origin xyz="0 0.0 -0.03" rpy="0 0 0"/>
+    <origin xyz="0 0.0 0" rpy="0 0 0"/>
     <parent link="right_arm_link5"/>
     <child link="right_arm_link6"/>
-    <axis xyz="0 -1 0" />
+    <axis xyz="1 0 0" />
     <dynamics damping ="0.1" />
     <limit effort="6.0" velocity="3.0" lower="-1.4" upper="1.57"/>
   </joint>
   <joint name="ra_7_joint" type="revolute">
-    <origin xyz="0 0.0 -0.055" rpy="0 0 0"/>
+    <origin xyz="0 0.0 -0.08" rpy="0 0 0"/>
     <parent link="right_arm_link6"/>
     <child link="right_arm_link7"/>

Commit message: Correct files for practice 09

File: catkin_ws/src/hardware/justina_description/urdf/justina_right_arm.xacro (robot description, xacro)
@@ -116,11 +116,4 @@
       <material name = "ra_material_blue"><color rgba="0 0 1 1"/></material>
     </visual>
-    <!--<visual>
-      <origin xyz="-0.01 0 -0.167" rpy = "0 0 0"/>
-      <geometry>
-        <box size = "0.06 -0.04025 0.04025"/>
-      </geometry>
-      <material name = "la_material_blue"><color rgba="0 0 1 1"/></material>
-    </visual> -->
     <collision>
       <origin xyz="0 0 -0.075" rpy = "0 0 0"/>
@@ -129,12 +122,6 @@
       </geometry>
     </collision>
-    <!--<collision>
-      <origin xyz="-0.01 0 -0.167" rpy = "0 0 0"/>
-      <geometry>
-        <box size = "0.06 0.04025 0.04025"/>
-      </geometry>
-    </collision> -->
-    <inertial>
-      <origin xyz="-0.01 0 -0.147" rpy = "0 0 0"/>
+    <inertial>
+      <origin xyz="0 0 -0.075" rpy = "0 0 0"/>
       <mass value="0.125"/>
       <inertia
@@ -159,5 +146,5 @@
     </collision>
     <inertial>
-      <origin xyz="0 0 -0.025" rpy = "0 0 0"/>
+      <origin xyz="0.02 0 0.005" rpy = "0 0 0"/>
       <mass value="0.125"/>
       <inertia
@@ -195,5 +182,5 @@
     </collision>
     <inertial>
-      <origin xyz="0 0 -0.042" rpy = "0 0 0"/>
+      <origin xyz="0 0 -0.062" rpy = "0 0 0"/>
       <mass value="0.125"/>
       <inertia
@@ -204,11 +191,4 @@
   </link>
   <link name="right_arm_link7">
-   <!-- <visual>
-      <origin xyz="-0.025 0 -0.03" rpy = "0 0 0"/>
-      <geometry>
-        <box size = "0.11 0.03525 0.03525"/>
-      </geometry>
-      <material name = "ra_material_or"><color rgba="1 0.5 0 1"/></material>
-    </visual>-->
     <visual>
       <origin xyz="0 0 -0.055" rpy = "0 0 0"/>
@@ -218,10 +198,4 @@
       <material name = "ra_material_green"><color rgba="0 0.5 0 1"/></material>
     </visual>
-    <!--<collision>
-      <origin xyz="-0.01 0 -0.03" rpy = "0 0 0"/>
-      <geometry>
-        <box size = "0.06 0.03525 0.03525"/>
-      </geometry>
-    </collision>-->
     <collision>
       <origin xyz="0 0 -0.055" rpy = "0 0 0"/>
@@ -231,5 +205,5 @@
     </collision>
     <inertial>
-      <origin xyz="-0.01 0 -0.05" rpy = "0 0 0"/>
+      <origin xyz="0 0 -0.055" rpy = "0 0 0"/>
       <mass value="0.125"/>
       <inertia

Commit message: Some changes in xacro files

File: catkin_ws/src/hardware/justina_description/urdf/justina_right_arm.xacro (robot description, xacro)
@@ -265,5 +265,5 @@
     <child link="right_arm_link1"/>
     <axis xyz="0 -1 0" />
-    <dynamics damping ="0.1" />
+    <dynamics damping ="0.1" friction="0.01"/>
     <limit effort="16.0" velocity="3.0" lower="-1.7" upper="1.7"/>
   </joint>
@@ -273,5 +273,5 @@
     <child link="right_arm_link2"/>
     <axis xyz="1 0 0" />
-    <dynamics damping ="0.1" />
+    <dynamics damping ="0.1" friction="0.01"/>
     <limit effort="8.0" velocity="3.0" lower="-1.85" upper="0.75"/>
   </joint>
@@ -281,5 +281,5 @@
     <child link="right_arm_link3"/>
     <axis xyz="0 0 1" />
-    <dynamics damping ="0.1" />
+    <dynamics damping ="0.1" friction="0.01"/>
     <limit effort="6.0" velocity="3.0" lower="-2.5" upper="2.5"/>
   </joint>
@@ -289,5 +289,5 @@
     <child link="right_arm_link4"/>
     <axis xyz="0 -1 0" />
-    <dynamics damping ="0.1" />
+    <dynamics damping ="0.1" friction="0.01"/>
     <limit effort="8.0" velocity="3.0" lower="-1.8" upper="1.8"/>
   </joint>
@@ -297,5 +297,5 @@
     <child link="right_arm_link5"/>
     <axis xyz="0 -1 0" />
-    <dynamics damping ="0.1" />
+    <dynamics damping ="0.1" friction="0.01"/>
     <limit effort="6.0" velocity="3.0" lower="-2.5" upper="2.5"/>
   </joint>
@@ -305,5 +305,5 @@
     <child link="right_arm_link6"/>
     <axis xyz="1 0 0" />
-    <dynamics damping ="0.1" />
+    <dynamics damping ="0.1" friction="0.01"/>
     <limit effort="6.0" velocity="3.0" lower="-1.4" upper="1.57"/>
   </joint>
@@ -313,5 +313,5 @@
     <child link="right_arm_link7"/>
     <axis xyz="0 0 1" />
-    <dynamics damping ="0.1" />
+    <dynamics damping ="0.1" friction="0.01"/>
     <limit effort="3.0" velocity="3.0" lower="-2.5" upper="2.5"/>
   </joint>
@@ -321,5 +321,5 @@
     <child link="right_arm_grip_left"/>
     <axis xyz="1 0 0" />
-    <dynamics damping ="0.1" />
+    <dynamics damping ="0.1" friction="0.01"/>
     <limit effort="3.0" velocity="3.0" lower="-0.3" upper="1.5"/>
   </joint>
@@ -329,5 +329,5 @@
     <child link="right_arm_grip_right"/>
     <axis xyz="-1 0 0" />
-    <dynamics damping ="0.1" />
+    <dynamics damping ="0.1" friction="0.01"/>
     <limit effort="3.0" velocity="3.0" lower="-0.3" upper="1.5"/>
   </joint>
